File: HW/discharger.kicad_pcb (KiCad board)
At the start: 2 copper layers, 87.2 x 73.7 mm, 85 parts, among them J1 Vin, J2 OLED, J3 Batt1, J4 Batt1, J5 Batt1, Q1 IRFFR220N, Q2 IRFFR220N, Q3 IRFFR220N, Q4 IRF7341, Q5 IRF7341, Q6 IRF7341, U1 LM2937, U10 MCP4728, U11 DW01-P, U12 DW01-P, U13 DW01-P, U2 LT1054, U3 INA219, U4 INA219, U5 OP07, U6 OP07, U7 INA219, U8 OP07, U9 ATMEGA328P-AU-Arduino, Y1 8MHZ

Commit message: grbl
Parts:
- moved C18 5.64 mm to (200.2, 103.4), turned to 90 degrees
- moved C20 5.23 mm to (200.3, 77.5), turned to 270 degrees
Routing:
- net Net-(C18-Pad2): track 24.6 -> 26.8 mm
- net Net-(C20-Pad2): track 21.6 -> 22.5 mm
Changed lines of the file:
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@@
 (kicad_pcb (version 4) (host pcbnew 4.0.7)
   (general
-    (links 216)
-    (no_connects 2)
+    (links 218)
+    (no_connects 0)
     (area 100.735001 62.650999 208.418501 147.226001)
     (thickness 1.6)
     (drawings 14)
-    (tracks 696)
+    (tracks 692)
     (zones 0)
     (modules 85)
@@
     (mod_text_size 1 1)
     (mod_text_width 0.15)
-    (pad_size 1.75 0.55)
-    (pad_drill 0)
+    (pad_size 3 3)
+    (pad_drill 1)
     (pad_to_mask_clearance 0.2)
     (aux_axis_origin 121.158 136.779)
     (visible_elements 7FFFEFFF)
     (pcbplotparams
-      (layerselection 0x01000_00000001)
+      (layerselection 0x010c0_80000001)
       (usegerberextensions false)
       (excludeedgelayer true)
@@
   )
   (module Capacitors_SMD:C_0805_HandSoldering (layer F.Cu)
-    (at 196.1388 99.5172)
+    (at 200.225 103.4 90)
     (descr "Capacitor SMD 0805, hand soldering")
     (tags "capacitor 0805")
     (attr smd)
-    (fp_text reference C18 (at 0 -1.75) (layer F.SilkS)
+    (fp_text reference C18 (at 0 -1.75 90) (layer F.SilkS)
       (effects (font (size 1 1) (thickness 0.15)))
     )
-    (fp_text value 22pf (at 0 1.75) (layer F.Fab)
+    (fp_text value 22pf (at 0 1.75 90) (layer F.Fab)
       (effects (font (size 1 1) (thickness 0.15)))
     )
-    (fp_text user %R (at 0 -1.75) (layer F.Fab)
+    (fp_text user %R (at 0 -1.75 90) (layer F.Fab)
       (effects (font (size 1 1) (thickness 0.15)))
     )
@@
     (fp_line (start 2.25 0.87) (end 2.25 -0.88) (layer F.CrtYd) (width 0.05))
     (fp_line (start 2.25 0.87) (end -2.25 0.87) (layer F.CrtYd) (width 0.05))
-    (pad 1 smd rect (at -1.25 0) (size 1.5 1.25) (layers F.Cu F.Paste F.Mask)
+    (pad 1 smd rect (at -1.25 0 90) (size 1.5 1.25) (layers F.Cu F.Paste F.Mask)
       (net 2 GND))
-    (pad 2 smd rect (at 1.25 0) (size 1.5 1.25) (layers F.Cu F.Paste F.Mask)
+    (pad 2 smd rect (at 1.25 0 90) (size 1.5 1.25) (layers F.Cu F.Paste F.Mask)
       (net 59 "Net-(C18-Pad2)"))
     (model Capacitors_SMD.3dshapes/C_0805.wrl
@@
   )
   (module Capacitors_SMD:C_0805_HandSoldering (layer F.Cu)
-    (at 196.5144 81.1276)
+    (at 200.325 77.55 270)
     (descr "Capacitor SMD 0805, hand soldering")
     (tags "capacitor 0805")
     (attr smd)
-    (fp_text reference C20 (at 0 -1.75) (layer F.SilkS)
+    (fp_text reference C20 (at 0 -1.75 270) (layer F.SilkS)
       (effects (font (size 1 1) (thickness 0.15)))
     )
-    (fp_text value 22pf (at 0 1.75) (layer F.Fab)
+    (fp_text value 22pf (at 0 1.75 270) (layer F.Fab)
       (effects (font (size 1 1) (thickness 0.15)))
     )
-    (fp_text user %R (at 0 -1.75) (layer F.Fab)
+    (fp_text user %R (at 0 -1.75 270) (layer F.Fab)
       (effects (font (size 1 1) (thickness 0.15)))
     )
@@
     (fp_line (start 2.25 0.87) (end 2.25 -0.88) (layer F.CrtYd) (width 0.05))
     (fp_line (start 2.25 0.87) (end -2.25 0.87) (layer F.CrtYd) (width 0.05))
-    (pad 1 smd rect (at -1.25 0) (size 1.5 1.25) (layers F.Cu F.Paste F.Mask)
+    (pad 1 smd rect (at -1.25 0 270) (size 1.5 1.25) (layers F.Cu F.Paste F.Mask)
       (net 2 GND))
-    (pad 2 smd rect (at 1.25 0) (size 1.5 1.25) (layers F.Cu F.Paste F.Mask)
+    (pad 2 smd rect (at 1.25 0 270) (size 1.5 1.25) (layers F.Cu F.Paste F.Mask)
       (net 61 "Net-(C20-Pad2)"))
     (model Capacitors_SMD.3dshapes/C_0805.wrl
@@
     (fp_line (start 7.79 -4) (end 7.79 4) (layer B.CrtYd) (width 0.05))
     (fp_line (start 7.79 -4) (end -2.71 -4) (layer B.CrtYd) (width 0.05))
-    (pad 1 thru_hole rect (at 0 0 90) (size 3 3) (drill 1.52) (layers *.Cu *.Mask)
+    (pad 1 thru_hole rect (at 0 0 90) (size 3 3) (drill 1) (layers *.Cu *.Mask)
       (net 2 GND))
-    (pad 2 thru_hole circle (at 5.08 0 90) (size 3 3) (drill 1.52) (layers *.Cu *.Mask)
+    (pad 2 thru_hole circle (at 5.08 0 90) (size 3 3) (drill 1) (layers *.Cu *.Mask)
       (net 9 "Net-(C4-Pad1)"))
     (model ${KISYS3DMOD}/Terminal_Blocks.3dshapes/TerminalBlock_bornier-2_P5.08mm.wrl
@@
     (fp_line (start 7.79 -4) (end 7.79 4) (layer B.CrtYd) (width 0.05))
     (fp_line (start 7.79 -4) (end -2.71 -4) (layer B.CrtYd) (width 0.05))
-    (pad 1 thru_hole rect (at 0 0 270) (size 3 3) (drill 1.52) (layers *.Cu *.Mask)
+    (pad 1 thru_hole rect (at 0 0 270) (size 3 3) (drill 1) (layers *.Cu *.Mask)
       (net 63 "Net-(C21-Pad2)"))
-    (pad 2 thru_hole circle (at 5.08 0 270) (size 3 3) (drill 1.52) (layers *.Cu *.Mask)
+    (pad 2 thru_hole circle (at 5.08 0 270) (size 3 3) (drill 1) (layers *.Cu *.Mask)
       (net 28 "/Battery connections/BatteryPositive1"))
     (model ${KISYS3DMOD}/Terminal_Blocks.3dshapes/TerminalBlock_bornier-2_P5.08mm.wrl
@@
     (fp_line (start 7.79 -4) (end 7.79 4) (layer B.CrtYd) (width 0.05))
     (fp_line (start 7.79 -4) (end -2.71 -4) (layer B.CrtYd) (width 0.05))
-    (pad 1 thru_hole rect (at 0 0 270) (size 3 3) (drill 1.52) (layers *.Cu *.Mask)
+    (pad 1 thru_hole rect (at 0 0 270) (size 3 3) (drill 1) (layers *.Cu *.Mask)
       (net 64 "Net-(C22-Pad2)"))
-    (pad 2 thru_hole circle (at 5.08 0 270) (size 3 3) (drill 1.52) (layers *.Cu *.Mask)
+    (pad 2 thru_hole circle (at 5.08 0 270) (size 3 3) (drill 1) (layers *.Cu *.Mask)
       (net 30 "/Battery connections/BatteryPositive2"))
     (model ${KISYS3DMOD}/Terminal_Blocks.3dshapes/TerminalBlock_bornier-2_P5.08mm.wrl
@@
     (fp_line (start 7.79 -4) (end 7.79 4) (layer B.CrtYd) (width 0.05))
     (fp_line (start 7.79 -4) (end -2.71 -4) (layer B.CrtYd) (width 0.05))
-    (pad 1 thru_hole rect (at 0 0) (size 3 3) (drill 1.52) (layers *.Cu *.Mask)
+    (pad 1 thru_hole rect (at 0 0) (size 3 3) (drill 1) (layers *.Cu *.Mask)
       (net 13 "Net-(C23-Pad2)"))
-    (pad 2 thru_hole circle (at 5.08 0) (size 3 3) (drill 1.52) (layers *.Cu *.Mask)
+    (pad 2 thru_hole circle (at 5.08 0) (size 3 3) (drill 1) (layers *.Cu *.Mask)
       (net 29 "/Battery connections/BatteryPositive3"))
     (model ${KISYS3DMOD}/Terminal_Blocks.3dshapes/TerminalBlock_bornier-2_P5.08mm.wrl
@@
   (segment (start 154.432 73.533) (end 152.93 73.533) (width 0.4) (layer B.Cu) (net 58))
   (segment (start 151.13 73.511) (end 151.13 73.386) (width 0.4) (layer B.Cu) (net 58))
+  (segment (start 200.225 102.15) (end 200.225 96.5869) (width 0.4) (layer F.Cu) (net 59))
+  (segment (start 200.225 96.5869) (end 200.0504 96.4123) (width 0.4) (layer F.Cu) (net 59))
   (segment (start 196.417093 88.171859) (end 195.667094 87.42186) (width 0.4) (layer F.Cu) (net 59))
   (segment (start 200.0504 96.4123) (end 200.0504 91.805166) (width 0.4) (layer F.Cu) (net 59))
@@
   (via (at 195.667094 87.42186) (size 1.5) (drill 0.8) (layers F.Cu B.Cu) (net 59))
   (segment (start 200.0504 91.805166) (end 196.417093 88.171859) (width 0.4) (layer F.Cu) (net 59))
-  (segment (start 200.0504 98.6536) (end 199.1868 99.5172) (width 0.4) (layer F.Cu) (net 59))
-  (segment (start 199.1868 99.5172) (end 197.3888 99.5172) (width 0.4) (layer F.Cu) (net 59))
   (segment (start 200.0504 96.4123) (end 200.0504 98.6536) (width 0.4) (layer F.Cu) (net 59))
-  (segment (start 197.5138 99.5172) (end 197.717 99.7204) (width 0.4) (layer F.Cu) (net 59))
-  (segment (start 197.3888 99.5172) (end 197.5138 99.5172) (width 0.4) (layer F.Cu) (net 59))
-  (segment (start 197.5138 99.5172) (end 197.6154 99.6188) (width 0.4) (layer F.Cu) (net 59))
   (segment (start 200.0504 95.0578) (end 200.0504 96.4123) (width 0.4) (layer F.Cu) (net 59))
   (segment (start 194.522372 102.328728) (end 194.522372 105.420828) (width 0.4) (layer B.Cu) (net 60))
   (segment (start 194.522372 105.420828) (end 194.3608 105.5824) (width 0.4) (layer B.Cu) (net 60))
+  (segment (start 200.325 78.8) (end 200.325 84.2627) (width 0.4) (layer F.Cu) (net 61))
+  (segment (start 200.325 84.2627) (end 200.0504 84.5373) (width 0.4) (layer F.Cu) (net 61))
   (segment (start 196.922372 93.828728) (end 196.953957 93.797143) (width 0.4) (layer B.Cu) (net 61))
   (segment (start 196.953957 93.797143) (end 196.953957 86.381417) (width 0.4) (layer B.Cu) (net 61))
@@
   (via (at 194.544511 83.971971) (size 1.5) (drill 0.8) (layers F.Cu B.Cu) (net 61))
   (segment (start 200.0504 84.5373) (end 195.10984 84.5373) (width 0.4) (layer F.Cu) (net 61))
-  (segment (start 197.7644 81.1276) (end 198.9144 81.1276) (width 0.4) (layer F.Cu) (net 61))
-  (segment (start 198.9144 81.1276) (end 200.0504 82.2636) (width 0.4) (layer F.Cu) (net 61))
-  (segment (start 200.0504 82.2636) (end 200.0504 84.5373) (width 0.4) (layer F.Cu) (net 61))
   (segment (start 132.06 99.949) (end 132.06 97.509) (width 0.4) (layer F.Cu) (net 62))
   (segment (start 132.06 97.509) (end 132.16 97.409) (width 0.4) (layer F.Cu) (net 62))

Commit message: better layout
Parts:
- removed the 1U1 at (193.7, 89.1)
- removed the 1U1 at (198.2, 106.5)
- removed C1: 2uF, Capacitors_SMD:C_0805_HandSoldering
- removed C11, C12, C15: 100n, Capacitors_SMD:C_0805_HandSoldering
- removed C2: 10uF, Capacitors_Tantalum_SMD:CP_Tantalum_Case-C_EIA-6032-28_Hand
- removed C5: 2nF, Capacitors_SMD:C_0805_HandSoldering
- removed C6: 100uF, Capacitors_THT:CP_Radial_D6.3mm_P2.50mm
- removed R1: 20K, Resistors_SMD:R_0805_HandSoldering
- removed R2: 102.6K, Resistors_SMD:R_0805_HandSoldering
- removed U2: LT1054, Housings_DIP:DIP-8_W7.62mm_LongPads
- added 1U1: 0,1U, Capacitors_SMD:C_0805_HandSoldering, F.Cu at (256.2, 92.8)
- added 1U3: 0,1U, Capacitors_SMD:C_0805_HandSoldering, F.Cu at (237.9, 118.3)
- added 1U4: 0,1U, Capacitors_SMD:C_0805_HandSoldering, F.Cu at (256.2, 98.8)
- added C24: 100n, Capacitors_SMD:C_0805_HandSoldering, F.Cu at (132.6, 78.4)
- added C25: 100n, Capacitors_SMD:C_0805_HandSoldering, F.Cu at (144.4, 78.4)
- added C26: 1n, Capacitors_SMD:C_0805_HandSoldering, B.Cu at (130.2, 102.8)
- added C27: 1n, Capacitors_SMD:C_0805_HandSoldering, B.Cu at (145.3, 102.5)
- added C28: 100n, Capacitors_SMD:C_0805_HandSoldering, F.Cu at (157.3, 78.6)
- added C29: 1n, Capacitors_SMD:C_0805_HandSoldering, B.Cu at (160.2, 102.9)
- added ISP1: ISP-header, Pin_Headers:Pin_Header_Straight_2x03_Pitch2.54mm, F.Cu at (216.1, 117.5)
- added Q7: BC847, TO_SOT_Packages_SMD:SOT-23_Handsoldering, B.Cu at (157.8, 139.6)
- added Q8: BC847, TO_SOT_Packages_SMD:SOT-23_Handsoldering, B.Cu at (137.7, 140.2)
- added Q9: BC847, TO_SOT_Packages_SMD:SOT-23_Handsoldering, B.Cu at (128.1, 117.8)
- added R27: 10K, Resistors_SMD:R_0805_HandSoldering, F.Cu at (133.9, 118.0)
- added R28: 10K, Resistors_SMD:R_0805_HandSoldering, F.Cu at (134.0, 120.7)
- added R29: 1K, Resistors_SMD:R_0805_HandSoldering, B.Cu at (125.5, 102.8)
- added R30: 1K, Resistors_SMD:R_0805_HandSoldering, B.Cu at (140.4, 102.5)
- added R31: 10K, Resistors_SMD:R_0805_HandSoldering, F.Cu at (134.1, 123.7)
- added R32: 1K, Resistors_SMD:R_0805_HandSoldering, B.Cu at (155.3, 102.9)
- added R33: 100R, Resistors_SMD:R_0805_HandSoldering, B.Cu at (158.7, 145.5)
- added R34: 100R, Resistors_SMD:R_0805_HandSoldering, B.Cu at (140.8, 143.1)
- added R35: 100R, Resistors_SMD:R_0805_HandSoldering, B.Cu at (129.4, 123.8)
- 1U2, C16, C17, C19, J1, J3, R12, R13, R14, R15, R16, R17, R18, R19, R20, R9: moved to F.Cu
- C21, C22, C23, Q4, Q5, Q6, R21, R22, R23, R24, R25, R26, U11, U12, U13: moved to B.Cu
- J4: value Batt1 -> Batt2; moved to F.Cu
- J5: value Batt1 -> Batt3; moved to F.Cu
- R5, R6, R8: footprint Resistors_THT:R_Axial_DIN0414_L11.9mm_D4.5mm_P15.24mm_Horizontal -> Resistors_SMD:R_2512_HandSoldering; moved to B.Cu
- U10: footprint Peter:MCP4728_on_a_breadboard -> Housings_DIP:DIP-10_W7.62mm_LongPads; moved to F.Cu
- Y1: footprint Crystals:Crystal_SMD_HC49-SD_HandSoldering -> Crystals:Crystal_HC18-U_Vertical
- moved TP1 115.0 mm to (57.0, 119.4)
- moved TP2 102.7 mm to (75.0, 105.5)
- moved TP3 95.5 mm to (74.5, 110.3)
- moved R10 84.9 mm to (220.2, 99.8), turned to 90 degrees
- moved 1U2 83.1 mm to (261.5, 92.8)
- moved R11 82.8 mm to (223.1, 99.8)
- moved J5 66.8 mm to (155.6, 71.6), turned to 180 degrees
- moved D1 62.4 mm to (167.4, 126.7)
- moved D2 60.6 mm to (182.4, 127.0)
- moved C23 59.9 mm to (156.0, 76.3), turned to 0 degrees
- moved D3 58.3 mm to (174.4, 126.5)
- moved JP1 57.5 mm to (238.8, 93.4)
- moved C9 56.2 mm to (123.0, 117.7)
- moved R15 52.9 mm to (171.5, 121.2), turned to 90 degrees
- moved R18 52.6 mm to (169.3, 121.1), turned to 90 degrees
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Connections:
- net Net-(Q1-Pad1) renamed /Dynamic load/B1off
- net Net-(Q2-Pad1) renamed /Dynamic load/B2off
- net Net-(Q3-Pad1) renamed /Dynamic load/B3off
- Q4 pad 6: Net-(Q4-Pad5) -> (no net)
- Q4 pad 7: Net-(Q4-Pad5) -> (no net)
- Q5 pad 6: Net-(Q5-Pad5) -> (no net)
- Q5 pad 7: Net-(Q5-Pad5) -> (no net)
- Q6 pad 6: Net-(Q6-Pad5) -> (no net)
- Q6 pad 7: Net-(Q6-Pad5) -> (no net)
- U4 pad 7: SCL -> VCC
- U4 pad 8: GND -> VCC
- U5 pad 4: -5V -> GND
- U6 pad 4: -5V -> GND
- U8 pad 4: -5V -> GND
- U9 pad 23: (no net) -> Net-(R33-Pad2)
- U9 pad 24: (no net) -> Net-(R34-Pad2)
- U9 pad 25: (no net) -> Net-(R35-Pad2)
Routing:
- net VCC: track 401.5 -> 176.5 mm, vias 3 -> 0
- net -5V: track 96.5 -> 0.00 mm
- net SDA: track 152.4 -> 68.4 mm, vias 4 -> 2
- net SCL: track 155.5 -> 72.8 mm, vias 4 -> 0
- net /Dynamic load/DAC_IN2: track 71.1 -> 22.2 mm
- net GND: track 155.1 -> 117.2 mm, vias 3 -> 0
- net Led2G: track 30.6 -> 0.00 mm
- net Led2B: track 29.7 -> 0.00 mm
- net Led2R: track 29.3 -> 0.00 mm
- net Led1G: track 28.4 -> 0.00 mm
- net Led1B: track 27.0 -> 0.00 mm
- net Led1R: track 26.8 -> 0.00 mm
- net Net-(C18-Pad2): track 26.8 -> 0.00 mm, vias 1 -> 0
- net Net-(C4-Pad1): track 24.7 -> 0.00 mm
- net reset_in: track 24.4 -> 0.00 mm
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Other:
- board size 87.2 x 73.7 mm -> 69.9 x 69.9 mm
- net class Batt+: clearance 0.4 -> 0.2
- net class Default: clearance 0.2 -> 0.25
- rule trace_clearance: 0.2 -> 0.25
