File: HW/discharger.kicad_pcb (KiCad board)
At the start: 2 copper layers, 69.9 x 69.9 mm, 95 parts, among them J1 Vin, J2 OLED, J3 Batt1, J4 Batt2, J5 Batt3, Q1 IRFFR220N, Q2 IRFFR220N, Q3 IRFFR220N, Q4 IRF7341, Q5 IRF7341, Q6 IRF7341, Q7 BC847, Q8 BC847, Q9 BC847, U1 LM2937, U10 MCP4728, U11 DW01-P, U12 DW01-P, U13 DW01-P, U3 INA219, U4 INA219, U5 OP07, U6 OP07, U7 INA219, U8 OP07, U9 ATMEGA328P-AU-Arduino, Y1 8MHZ

Commit message: Layout complete
Done
Parts:
- removed ISP1: ISP-header, Pin_Headers:Pin_Header_Straight_2x03_Pitch2.54mm
- removed TP1, TP2, TP3: TEST, Pin_Headers:Pin_Header_Straight_1x01_Pitch2.54mm
- 1U1, 1U2, 1U3, 1U4, C10, C16, C17, C18, C19, C20, R10, R11, R12, R13, R14, R15, R16, R17, R18, R19, R20, R9: moved to B.Cu
- J2: footprint Pin_Headers:Pin_Header_Straight_1x04_Pitch2.54mm_SMD_Pin1Left -> Pin_Headers:Pin_Header_Straight_1x04_Pitch2.54mm
- moved 1U2 100.4 mm to (161.2, 87.4), turned to 90 degrees
- moved 1U1 82.3 mm to (174.3, 101.3), turned to 90 degrees
- moved 1U4 76.7 mm to (182.2, 119.2), turned to 270 degrees
- moved C20 65.9 mm to (172.8, 121.8), turned to 90 degrees
- moved R10 59.5 mm to (161.2, 93.0), turned to 270 degrees
- moved 1U3 57.7 mm to (180.2, 119.2), turned to 270 degrees
- moved C19 56.7 mm to (178.4, 101.3), turned to 90 degrees
- moved C18 56.4 mm to (177.8, 121.7), turned to 90 degrees
- moved R11 55.1 mm to (168.5, 92.0), turned to 270 degrees
- moved Y1 51.7 mm to (177.7, 118.0), turned to 180 degrees
- moved JP1 51.3 mm to (189.0, 81.1)
- moved R33 28.8 mm to (161.9, 116.8), turned to 0 degrees
- moved R16 28.6 mm to (159.2, 126.9)
- moved C17 26.8 mm to (186.8, 91.1), turned to 90 degrees
- moved Q7 24.4 mm to (156.9, 115.2)
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Connections:
- R33 pad 2: Net-(R33-Pad2) -> B3off_MCU
- R34 pad 2: Net-(R34-Pad2) -> B2off_MCU
- R35 pad 2: Net-(R35-Pad2) -> B1off_MCU
- U9 pad 15: MOSI -> B1off_MCU
- U9 pad 16: MISO -> B2off_MCU
- U9 pad 17: SCK -> B3off_MCU
- U9 pad 23: Net-(R33-Pad2) -> (no net)
- U9 pad 24: Net-(R34-Pad2) -> (no net)
- U9 pad 25: Net-(R35-Pad2) -> (no net)
Routing:
- net GND: track 117.2 -> 627.4 mm
- net VCC: track 176.5 -> 447.9 mm, vias 0 -> 1
- net SDA: track 68.4 -> 177.2 mm, vias 2 -> 4
- net SCL: track 72.8 -> 175.7 mm, vias 0 -> 1
- net B1off_MCU: track 0.00 -> 68.3 mm
- net B2off_MCU: track 0.00 -> 61.0 mm
- net reset_in: track 0.00 -> 49.1 mm, vias 0 -> 1
- net Led2G: track 0.00 -> 26.5 mm
- net RXI: track 0.00 -> 25.0 mm
- net TX0: track 0.00 -> 24.6 mm
- net Led2B: track 0.00 -> 23.9 mm
- net Led2R: track 0.00 -> 21.5 mm
- net B3off_MCU: track 0.00 -> 20.2 mm
- net Led1G: track 0.00 -> 19.2 mm
- net Led1B: track 0.00 -> 17.7 mm
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Other:
- board text added: "-VIN+"
- board text removed: "B1"
- board text removed: "B2"
- board text removed: "B3"
