File: HW/discharger.sch (KiCad schematic (older format))
At the start: 0 parts

Commit message: Add files via upload
Changed lines of the file:
@@
 $Descr A4 11693 8268
 encoding utf-8
-Sheet 1 4
+Sheet 1 5
 Title ""
 Date ""
@@
 F0 "Dynamic load" 60
 F1 "Current gen.sch" 60
+F2 "Battery_Positive1" I R 7000 2250 60
+F3 "Battery_Positive3" I R 7000 2500 60
+F4 "Battery_Positive2" I R 7000 2375 60
 $EndSheet
 $Sheet
@@
 F1 "mcu.sch" 60
 $EndSheet
+$Sheet
+S 4950 3600 2050 1400
+U 5A978CF2
+F0 "Battery connections" 60
+F1 "Batteries.sch" 60
+F2 "BatteryPositive1" I R 7000 3750 60
+F3 "BatteryPositive3" I R 7000 4000 60
+F4 "BatteryPositive2" I R 7000 3875 60
+$EndSheet
+Wire Wire Line
+	7000 2250 7500 2250
+Wire Wire Line
+	7500 2250 7500 3750
+Wire Wire Line
+	7500 3750 7000 3750
+Wire Wire Line
+	7000 3875 7425 3875
+Wire Wire Line
+	7425 3875 7425 2375
+Wire Wire Line
+	7425 2375 7000 2375
+Wire Wire Line
+	7000 2500 7325 2500
+Wire Wire Line
+	7325 2500 7325 4000
+Wire Wire Line
+	7325 4000 7000 4000
 $EndSCHEMATC

Commit message: Add files via upload
Changed lines of the file:
@@
 LIBS:contrib
 LIBS:valves
-LIBS:3-pin-boostconv
-LIBS:34063
-LIBS:Arduino
-LIBS:bluepill_breakouts
-LIBS:L298N
-LIBS:Peter-bckup
-LIBS:Peters
-LIBS:WS2812B
 LIBS:discharger-cache
 EELAYER 25 0
@@
 $EndDescr
 $Sheet
-S 1900 3600 2150 1400
+S 1450 3500 2150 1400
 U 5A970EC9
 F0 "PSU" 60
@@
 F3 "Battery_Positive3" I R 7000 2500 60
 F4 "Battery_Positive2" I R 7000 2375 60
+F5 "BattV_Monitor3" I L 4950 2700 60
+F6 "BattV_Monitor2" I L 4950 2800 60
+F7 "DAC_IN1" I L 4950 1950 60
+F8 "BattV_Monitor1" I L 4950 2900 60
+F9 "DAC_IN3" I L 4950 2150 60
+F10 "DAC_IN2" I L 4950 2050 60
 $EndSheet
 $Sheet
-S 1450 1550 2600 1350
+S 1400 1550 2600 1350
 U 5A970EED
 F0 "MCU" 60
 F1 "mcu.sch" 60
+F2 "DAC_OUT1" I R 4000 1950 60
+F3 "DAC_OUT2" I R 4000 2050 60
+F4 "DAC_OUT3" I R 4000 2150 60
 $EndSheet
 $Sheet
@@
 Wire Wire Line
 	7325 4000 7000 4000
+Wire Wire Line
+	4000 1950 4950 1950
+Wire Wire Line
+	4000 2050 4950 2050
+Wire Wire Line
+	4000 2150 4950 2150
 $EndSCHEMATC

Commit message: better layout
Changed lines of the file:
@@
 F3 "Battery_Positive3" I R 7000 2500 60
 F4 "Battery_Positive2" I R 7000 2375 60
-F5 "BattV_Monitor3" I L 4950 2700 60
-F6 "BattV_Monitor2" I L 4950 2800 60
-F7 "DAC_IN1" I L 4950 1950 60
-F8 "BattV_Monitor1" I L 4950 2900 60
-F9 "DAC_IN3" I L 4950 2150 60
-F10 "DAC_IN2" I L 4950 2050 60
+F5 "DAC_IN1" I L 4950 1950 60
+F6 "DAC_IN3" I L 4950 2150 60
+F7 "DAC_IN2" I L 4950 2050 60
+F8 "B1off" I L 4950 2500 60
+F9 "B2off" I L 4950 2600 60
+F10 "B3off" I L 4950 2700 60
 $EndSheet
 $Sheet
@@
 F3 "DAC_OUT2" I R 4000 2050 60
 F4 "DAC_OUT3" I R 4000 2150 60
+F5 "B1off" I R 4000 2500 60
+F6 "B2off" I R 4000 2600 60
+F7 "B3off" I R 4000 2700 60
 $EndSheet
 $Sheet
@@
 Wire Wire Line
 	4000 2150 4950 2150
+Wire Wire Line
+	4000 2500 4950 2500
+Wire Wire Line
+	4000 2600 4950 2600
+Wire Wire Line
+	4000 2700 4950 2700
 $EndSCHEMATC
