File: HW/power.sch (KiCad schematic (older format))
At the start: 0 parts

Commit message: Add files via upload
Parts:
- added C?: 10uF, symbol CP_Small
- added C?: 2uF, symbol C_Small
- added C?: 100uF, symbol CP_Small
- added C?: 2nF, symbol C_Small
- added R?: 20K, symbol R
- added R?: 102.6K, symbol R
- added U?: LT1054, Housings_DIP:DIP-8_W7.62mm_LongPads, symbol LT1054
Connections:
- new net: C?.1, R?.1, R?.1, U?.1 (FB/SD)
- new net: C?.1, U?.2 (CAP+)
- new net: C?.2, U?.4 (CAP-)
- new net: R?.2, U?.6 (VREF)
- new net -5V: C?.2, C?.2, R?.2, U?.5 (VOUT)
- new net GND: C?.1, C?.2, U?.3 (GND)
- new net VCC: C?.1, U?.8 (VCC)
Changed lines of the file:
@@
 $Descr A4 11693 8268
 encoding utf-8
-Sheet 1 4
+Sheet 2 5
 Title ""
 Date ""
@@
 Comment4 ""
 $EndDescr
+$Comp
+L -5V #PWR?
+U 1 1 5A971C8A
+P 4050 3500
+F 0 "#PWR?" H 4050 3600 50  0001 C CNN
+F 1 "-5V" H 4050 3650 50  0000 C CNN
+F 2 "" H 4050 3500 50  0001 C CNN
+F 3 "" H 4050 3500 50  0001 C CNN
+	1    4050 3500
+	1    0    0    -1
+$EndComp
+$Comp
+L LT1054 U?
+U 1 1 5A971C9E
+P 2650 3200
+F 0 "U?" H 2350 3700 60  0000 C CNN
+F 1 "LT1054" H 2350 3050 60  0000 C CNN
+F 2 "Housings_DIP:DIP-8_W7.62mm_LongPads" H 2850 2750 60  0001 C CNN
+F 3 "http://www.ti.com/lit/ds/symlink/lt1054.pdf" H 3000 2850 60  0001 C CNN
+	1    2650 3200
+	1    0    0    -1
+$EndComp
+$Comp
+L GND #PWR01
+U 1 1 5A971D46
+P 2650 3500
+F 0 "#PWR01" H 2650 3250 50  0001 C CNN
+F 1 "GND" H 2650 3350 50  0000 C CNN
+F 2 "" H 2650 3500 50  0001 C CNN
+F 3 "" H 2650 3500 50  0001 C CNN
+	1    2650 3500
+	1    0    0    -1
+$EndComp
+Wire Wire Line
+	2650 3450 2650 3500
+$Comp
+L CP_Small C?
+U 1 1 5A971DAC
+P 1900 3100
+F 0 "C?" H 1910 3170 50  0000 L CNN
+F 1 "10uF" V 1800 3000 50  0000 L CNN
+F 2 "" H 1900 3100 50  0001 C CNN
+F 3 "" H 1900 3100 50  0001 C CNN
+	1    1900 3100
+	1    0    0    -1
+$EndComp
+Wire Wire Line
+	2100 3000 1900 3000
+Wire Wire Line
+	2100 3100 2100 3200
+Wire Wire Line
+	2100 3200 1900 3200
+$Comp
+L R R?
+U 1 1 5A971E49
+P 3500 3000
+F 0 "R?" V 3400 3000 50  0000 C CNN
+F 1 "20K" V 3500 3000 50  0000 C CNN
+F 2 "" V 3430 3000 50  0001 C CNN
+F 3 "" H 3500 3000 50  0001 C CNN
+	1    3500 3000
+	0    1    1    0
+$EndComp
+Wire Wire Line
+	3350 3000 3150 3000
+$Comp
+L VCC #PWR02
+U 1 1 5A971ED5
+P 2650 2250
+F 0 "#PWR02" H 2650 2100 50  0001 C CNN
+F 1 "VCC" H 2650 2400 50  0000 C CNN
+F 2 "" H 2650 2250 50  0001 C CNN
+F 3 "" H 2650 2250 50  0001 C CNN
+	1    2650 2250
+	1    0    0    -1
+$EndComp
+$Comp
+L C_Small C?
+U 1 1 5A971F06
+P 2800 2400
+F 0 "C?" H 2810 2470 50  0000 L CNN
+F 1 "2uF" H 2810 2320 50  0000 L CNN
+F 2 "" H 2800 2400 50  0001 C CNN
+F 3 "" H 2800 2400 50  0001 C CNN
+	1    2800 2400
+	1    0    0    -1
+$EndComp
+$Comp
+L GND #PWR03
+U 1 1 5A971F51
+P 2800 2500
+F 0 "#PWR03" H 2800 2250 50  0001 C CNN
+F 1 "GND" H 2800 2350 50  0000 C CNN
+F 2 "" H 2800 2500 50  0001 C CNN
+F 3 "" H 2800 2500 50  0001 C CNN
+	1    2800 2500
+	1    0    0    -1
+$EndComp
+Wire Wire Line
+	2650 2250 2650 2300
+Wire Wire Line
+	2650 2300 2650 2600
+Wire Wire Line
+	2800 2300 2650 2300
+Connection ~ 2650 2300
+$Comp
+L R R?
+U 1 1 5A971FF1
+P 3500 3100
+F 0 "R?" V 3580 3100 50  0000 C CNN
+F 1 "102.6K" V 3500 3100 50  0000 C CNN
+F 2 "" V 3430 3100 50  0001 C CNN
+F 3 "" H 3500 3100 50  0001 C CNN
+	1    3500 3100
+	0    1    1    0
+$EndComp
+Wire Wire Line
+	3150 3100 3200 3100
+Wire Wire Line
+	3200 3100 3350 3100
+Wire Wire Line
+	2100 2900 2100 2050
+Wire Wire Line
+	2100 2050 3650 2050
+Wire Wire Line
+	3650 2050 3650 3000
+Wire Wire Line
+	3650 3000 3650 3100
+Wire Wire Line
+	3650 3100 3650 3350
+Connection ~ 3650 3000
+Wire Wire Line
+	3200 3100 3200 3550
+Wire Wire Line
+	3200 3550 3650 3550
+Wire Wire Line
+	3650 3550 4050 3550
+Connection ~ 3200 3100
+$Comp
+L CP_Small C?
+U 1 1 5A9720FC
+P 3200 3650
+F 0 "C?" H 3210 3720 50  0000 L CNN
+F 1 "100uF" H 3210 3570 50  0000 L CNN
+F 2 "" H 3200 3650 50  0001 C CNN
+F 3 "" H 3200 3650 50  0001 C CNN
+	1    3200 3650
+	-1   0    0    1
+$EndComp
+$Comp
+L GND #PWR04
+U 1 1 5A972177
+P 3200 3800
+F 0 "#PWR04" H 3200 3550 50  0001 C CNN
+F 1 "GND" H 3200 3650 50  0000 C CNN
+F 2 "" H 3200 3800 50  0001 C CNN
+F 3 "" H 3200 3800 50  0001 C CNN
+	1    3200 3800
+	1    0    0    -1
+$EndComp
+Wire Wire Line
+	3200 3800 3200 3750
+Wire Wire Line
+	4050 3550 4050 3500
+Connection ~ 3650 3100
+$Comp
+L C_Small C?
+U 1 1 5A97221D
+P 3650 3450
+F 0 "C?" H 3660 3520 50  0000 L CNN
+F 1 "2nF" H 3800 3450 50  0000 L CNN
+F 2 "" H 3650 3450 50  0001 C CNN
+F 3 "" H 3650 3450 50  0001 C CNN
+	1    3650 3450
+	1    0    0    -1
+$EndComp
+Connection ~ 3650 3550
 $EndSCHEMATC

Commit message: Add files via upload
Parts:
- C1: renamed from C?; footprint (none) -> Capacitors_Tantalum_SMD:CP_Tantalum_Case-C_EIA-6032-28_Hand
- C2, C4: renamed from C?; footprint (none) -> Capacitors_SMD:C_0805_HandSoldering
- C3: renamed from C?; footprint (none) -> Capacitors_THT:CP_Radial_D6.3mm_P2.50mm
- R1, R2: renamed from R?; footprint (none) -> Resistors_SMD:R_0805_HandSoldering
- gave numbers to parts that had none: 1
Changed lines of the file:
@@
 LIBS:Peters
 LIBS:WS2812B
-LIBS:pro-mini-cache
+LIBS:discharger-cache
 EELAYER 25 0
 EELAYER END
@@
 $EndDescr
 $Comp
-L -5V #PWR?
+L -5V #PWR5
 U 1 1 5A971C8A
 P 4050 3500
-F 0 "#PWR?" H 4050 3600 50  0001 C CNN
+F 0 "#PWR5" H 4050 3600 50  0001 C CNN
 F 1 "-5V" H 4050 3650 50  0000 C CNN
 F 2 "" H 4050 3500 50  0001 C CNN
@@
 $EndComp
 $Comp
-L LT1054 U?
+L LT1054 U1
 U 1 1 5A971C9E
 P 2650 3200
-F 0 "U?" H 2350 3700 60  0000 C CNN
+F 0 "U1" H 2350 3700 60  0000 C CNN
 F 1 "LT1054" H 2350 3050 60  0000 C CNN
 F 2 "Housings_DIP:DIP-8_W7.62mm_LongPads" H 2850 2750 60  0001 C CNN
@@
 $EndComp
 $Comp
-L GND #PWR01
+L GND #PWR2
 U 1 1 5A971D46
 P 2650 3500
-F 0 "#PWR01" H 2650 3250 50  0001 C CNN
+F 0 "#PWR2" H 2650 3250 50  0001 C CNN
 F 1 "GND" H 2650 3350 50  0000 C CNN
 F 2 "" H 2650 3500 50  0001 C CNN
@@
 	2650 3450 2650 3500
 $Comp
-L CP_Small C?
+L CP_Small C1
 U 1 1 5A971DAC
 P 1900 3100
-F 0 "C?" H 1910 3170 50  0000 L CNN
+F 0 "C1" H 1910 3170 50  0000 L CNN
 F 1 "10uF" V 1800 3000 50  0000 L CNN
-F 2 "" H 1900 3100 50  0001 C CNN
+F 2 "Capacitors_Tantalum_SMD:CP_Tantalum_Case-C_EIA-6032-28_Hand" H 1900 3100 50  0001 C CNN
 F 3 "" H 1900 3100 50  0001 C CNN
 	1    1900 3100
@@
 	2100 3200 1900 3200
 $Comp
-L R R?
+L R R1
 U 1 1 5A971E49
 P 3500 3000
-F 0 "R?" V 3400 3000 50  0000 C CNN
+F 0 "R1" V 3400 3000 50  0000 C CNN
 F 1 "20K" V 3500 3000 50  0000 C CNN
-F 2 "" V 3430 3000 50  0001 C CNN
+F 2 "Resistors_SMD:R_0805_HandSoldering" V 3430 3000 50  0001 C CNN
 F 3 "" H 3500 3000 50  0001 C CNN
 	1    3500 3000
@@
 	3350 3000 3150 3000
 $Comp
-L VCC #PWR02
+L VCC #PWR1
 U 1 1 5A971ED5
 P 2650 2250
-F 0 "#PWR02" H 2650 2100 50  0001 C CNN
+F 0 "#PWR1" H 2650 2100 50  0001 C CNN
 F 1 "VCC" H 2650 2400 50  0000 C CNN
 F 2 "" H 2650 2250 50  0001 C CNN
@@
 $EndComp
 $Comp
-L C_Small C?
+L C_Small C2
 U 1 1 5A971F06
 P 2800 2400
-F 0 "C?" H 2810 2470 50  0000 L CNN
+F 0 "C2" H 2810 2470 50  0000 L CNN
 F 1 "2uF" H 2810 2320 50  0000 L CNN
-F 2 "" H 2800 2400 50  0001 C CNN
+F 2 "Capacitors_SMD:C_0805_HandSoldering" H 2800 2400 50  0001 C CNN
 F 3 "" H 2800 2400 50  0001 C CNN
 	1    2800 2400
@@
 $EndComp
 $Comp
-L GND #PWR03
+L GND #PWR3
 U 1 1 5A971F51
 P 2800 2500
-F 0 "#PWR03" H 2800 2250 50  0001 C CNN
+F 0 "#PWR3" H 2800 2250 50  0001 C CNN
 F 1 "GND" H 2800 2350 50  0000 C CNN
 F 2 "" H 2800 2500 50  0001 C CNN
@@
 $EndComp
 Wire Wire Line
-	2650 2250 2650 2300
-Wire Wire Line
-	2650 2300 2650 2600
+	2650 2250 2650 2600
 Wire Wire Line
 	2800 2300 2650 2300
 Connection ~ 2650 2300
 $Comp
-L R R?
+L R R2
 U 1 1 5A971FF1
 P 3500 3100
-F 0 "R?" V 3580 3100 50  0000 C CNN
+F 0 "R2" V 3580 3100 50  0000 C CNN
 F 1 "102.6K" V 3500 3100 50  0000 C CNN
-F 2 "" V 3430 3100 50  0001 C CNN
+F 2 "Resistors_SMD:R_0805_HandSoldering" V 3430 3100 50  0001 C CNN
 F 3 "" H 3500 3100 50  0001 C CNN
 	1    3500 3100
@@
 $EndComp
 Wire Wire Line
-	3150 3100 3200 3100
-Wire Wire Line
-	3200 3100 3350 3100
+	3150 3100 3350 3100
 Wire Wire Line
 	2100 2900 2100 2050
@@
 	2100 2050 3650 2050
 Wire Wire Line
-	3650 2050 3650 3000
-Wire Wire Line
-	3650 3000 3650 3100
-Wire Wire Line
-	3650 3100 3650 3350
+	3650 2050 3650 3350
 Connection ~ 3650 3000
 Wire Wire Line
 	3200 3100 3200 3550
 Wire Wire Line
-	3200 3550 3650 3550
-Wire Wire Line
-	3650 3550 4050 3550
+	3200 3550 4050 3550
 Connection ~ 3200 3100
 $Comp
-L CP_Small C?
+L CP_Small C3
 U 1 1 5A9720FC
 P 3200 3650
-F 0 "C?" H 3210 3720 50  0000 L CNN
+F 0 "C3" H 3210 3720 50  0000 L CNN
 F 1 "100uF" H 3210 3570 50  0000 L CNN
-F 2 "" H 3200 3650 50  0001 C CNN
+F 2 "Capacitors_THT:CP_Radial_D6.3mm_P2.50mm" H 3200 3650 50  0001 C CNN
 F 3 "" H 3200 3650 50  0001 C CNN
 	1    3200 3650
@@
 $EndComp
 $Comp
-L GND #PWR04
+L GND #PWR4
 U 1 1 5A972177
 P 3200 3800
-F 0 "#PWR04" H 3200 3550 50  0001 C CNN
+F 0 "#PWR4" H 3200 3550 50  0001 C CNN
 F 1 "GND" H 3200 3650 50  0000 C CNN
 F 2 "" H 3200 3800 50  0001 C CNN
@@
 Connection ~ 3650 3100
 $Comp
-L C_Small C?
+L C_Small C4
 U 1 1 5A97221D
 P 3650 3450
-F 0 "C?" H 3660 3520 50  0000 L CNN
+F 0 "C4" H 3660 3520 50  0000 L CNN
 F 1 "2nF" H 3800 3450 50  0000 L CNN
-F 2 "" H 3650 3450 50  0001 C CNN
+F 2 "Capacitors_SMD:C_0805_HandSoldering" H 3650 3450 50  0001 C CNN
 F 3 "" H 3650 3450 50  0001 C CNN
 	1    3650 3450

Commit message: Add files via upload
Parts:
- added C7, C8: C, Capacitors_SMD:C_0805_HandSoldering, symbol C
Other:
- note added: "LM2937"
Changed lines of the file:
@@
 LIBS:contrib
 LIBS:valves
-LIBS:3-pin-boostconv
-LIBS:34063
-LIBS:Arduino
-LIBS:bluepill_breakouts
-LIBS:L298N
-LIBS:Peter-bckup
-LIBS:Peters
-LIBS:WS2812B
 LIBS:discharger-cache
 EELAYER 25 0
@@
 $EndDescr
 $Comp
-L -5V #PWR5
+L -5V #PWR6
 U 1 1 5A971C8A
 P 4050 3500
-F 0 "#PWR5" H 4050 3600 50  0001 C CNN
+F 0 "#PWR6" H 4050 3600 50  0001 C CNN
 F 1 "-5V" H 4050 3650 50  0000 C CNN
 F 2 "" H 4050 3500 50  0001 C CNN
@@
 $EndComp
 $Comp
-L GND #PWR2
+L GND #PWR01
 U 1 1 5A971D46
 P 2650 3500
-F 0 "#PWR2" H 2650 3250 50  0001 C CNN
+F 0 "#PWR01" H 2650 3250 50  0001 C CNN
 F 1 "GND" H 2650 3350 50  0000 C CNN
 F 2 "" H 2650 3500 50  0001 C CNN
@@
 	3350 3000 3150 3000
 $Comp
-L VCC #PWR1
+L VCC #PWR02
 U 1 1 5A971ED5
 P 2650 2250
-F 0 "#PWR1" H 2650 2100 50  0001 C CNN
+F 0 "#PWR02" H 2650 2100 50  0001 C CNN
 F 1 "VCC" H 2650 2400 50  0000 C CNN
 F 2 "" H 2650 2250 50  0001 C CNN
@@
 $EndComp
 $Comp
-L GND #PWR3
+L GND #PWR03
 U 1 1 5A971F51
 P 2800 2500
-F 0 "#PWR3" H 2800 2250 50  0001 C CNN
+F 0 "#PWR03" H 2800 2250 50  0001 C CNN
 F 1 "GND" H 2800 2350 50  0000 C CNN
 F 2 "" H 2800 2500 50  0001 C CNN
@@
 $EndComp
 $Comp
-L GND #PWR4
+L GND #PWR04
 U 1 1 5A972177
 P 3200 3800
-F 0 "#PWR4" H 3200 3550 50  0001 C CNN
+F 0 "#PWR04" H 3200 3550 50  0001 C CNN
 F 1 "GND" H 3200 3650 50  0000 C CNN
 F 2 "" H 3200 3800 50  0001 C CNN
@@
 $EndComp
 Connection ~ 3650 3550
+Text Notes 6300 2500 0    60   ~ 0
+LM2937
+$Comp
+L +5V #PWR05
+U 1 1 5A9EEEA2
+P 7050 2500
+F 0 "#PWR05" H 7050 2350 50  0001 C CNN
+F 1 "+5V" H 7050 2640 50  0000 C CNN
+F 2 "" H 7050 2500 50  0001 C CNN
+F 3 "" H 7050 2500 50  0001 C CNN
+	1    7050 2500
+	1    0    0    -1
+$EndComp
+$Comp
+L C C8
+U 1 1 5A9EEEC4
+P 5450 3050
+F 0 "C8" H 5475 3150 50  0000 L CNN
+F 1 "C" H 5475 2950 50  0000 L CNN
+F 2 "Capacitors_SMD:C_0805_HandSoldering" H 5488 2900 50  0001 C CNN
+F 3 "" H 5450 3050 50  0001 C CNN
+	1    5450 3050
+	1    0    0    -1
+$EndComp
+$Comp
+L C C7
+U 1 1 5A9EEF1F
+P 7800 3000
+F 0 "C7" H 7825 3100 50  0000 L CNN
+F 1 "C" H 7825 2900 50  0000 L CNN
+F 2 "Capacitors_SMD:C_0805_HandSoldering" H 7838 2850 50  0001 C CNN
+F 3 "" H 7800 3000 50  0001 C CNN
+	1    7800 3000
+	1    0    0    -1
+$EndComp
+$Comp
+L GND #PWR06
+U 1 1 5A9EEF79
+P 6700 3450
+F 0 "#PWR06" H 6700 3200 50  0001 C CNN
+F 1 "GND" H 6700 3300 50  0000 C CNN
+F 2 "" H 6700 3450 50  0001 C CNN
+F 3 "" H 6700 3450 50  0001 C CNN
+	1    6700 3450
+	1    0    0    -1
+$EndComp
 $EndSCHEMATC

Commit message: Add files via upload
Parts:
- added U?: LM2937, TO_SOT_Packages_SMD:SOT-223-3_TabPin2, symbol LM2937
Changed lines of the file:
@@
 LIBS:contrib
 LIBS:valves
+LIBS:3-pin-boostconv
+LIBS:34063
+LIBS:Arduino
+LIBS:bluepill_breakouts
+LIBS:L298N
+LIBS:Peter-bckup
+LIBS:Peters
+LIBS:WS2812B
 LIBS:discharger-cache
 EELAYER 25 0
@@
 	1    0    0    -1
 $EndComp
+$Comp
+L LM2937 U?
+U 1 1 5A9F8E30
+P 6650 2900
+F 0 "U?" H 6500 3000 60  0000 C CNN
+F 1 "LM2937" H 6550 2900 60  0000 C CNN
+F 2 "TO_SOT_Packages_SMD:SOT-223-3_TabPin2" H 6400 2900 60  0001 C CNN
+F 3 "http://www.ti.com/lit/ds/symlink/lm2937.pdf" H 6500 3000 60  0001 C CNN
+	1    6650 2900
+	1    0    0    -1
+$EndComp

Commit message: Add files via upload
Parts:
- added J1: Vin, Connectors_Terminal_Blocks:TerminalBlock_bornier-2_P5.08mm, symbol Screw_Terminal_01x02
- C3: renamed from C7; value C -> 10uF
- C4: renamed from C8; value C -> 0,1uF
- gave numbers to parts that had none: 1
- renumbered C2 to C1, C1 to C2, C4 to C5, C3 to C6, U1 to U2
Connections:
- net GND: now also C3.2, C4.2, U1.2 (GND), J1.1 (Pin_1)
- net VCC: now also C3.1, U1.3 (VOUT)
- net at C4.1: now also U1.1 (VIN), J1.2 (Pin_2)
Other:
- moved on the sheet: C3, C4

Commit message: better layout
Parts:
- removed C1: 2uF, Capacitors_SMD:C_0805_HandSoldering, symbol C_Small
- removed C2: 10uF, Capacitors_Tantalum_SMD:CP_Tantalum_Case-C_EIA-6032-28_Hand, symbol CP_Small
- removed C5: 2nF, Capacitors_SMD:C_0805_HandSoldering, symbol C_Small
- removed C6: 100uF, Capacitors_THT:CP_Radial_D6.3mm_P2.50mm, symbol CP_Small
- removed R1: 20K, Resistors_SMD:R_0805_HandSoldering, symbol R
- removed R2: 102.6K, Resistors_SMD:R_0805_HandSoldering, symbol R
- removed U2: LT1054, Housings_DIP:DIP-8_W7.62mm_LongPads, symbol LT1054
Changed lines of the file:
@@
 Comment4 ""
 $EndDescr
-$Comp
-L -5V #PWR6
-U 1 1 5A971C8A
-P 4050 3500
-F 0 "#PWR6" H 4050 3600 50  0001 C CNN
-F 1 "-5V" H 4050 3650 50  0000 C CNN
-F 2 "" H 4050 3500 50  0001 C CNN
-F 3 "" H 4050 3500 50  0001 C CNN
-	1    4050 3500
-	1    0    0    -1
-$EndComp
-$Comp
-L LT1054 U2
-U 1 1 5A971C9E
-P 2650 3200
-F 0 "U2" H 2350 3700 60  0000 C CNN
-F 1 "LT1054" H 2350 3050 60  0000 C CNN
-F 2 "Housings_DIP:DIP-8_W7.62mm_LongPads" H 2850 2750 60  0001 C CNN
-F 3 "http://www.ti.com/lit/ds/symlink/lt1054.pdf" H 3000 2850 60  0001 C CNN
-	1    2650 3200
-	1    0    0    -1
-$EndComp
-$Comp
-L GND #PWR01
-U 1 1 5A971D46
-P 2650 3500
-F 0 "#PWR01" H 2650 3250 50  0001 C CNN
-F 1 "GND" H 2650 3350 50  0000 C CNN
-F 2 "" H 2650 3500 50  0001 C CNN
-F 3 "" H 2650 3500 50  0001 C CNN
-	1    2650 3500
-	1    0    0    -1
-$EndComp
-Wire Wire Line
-	2650 3450 2650 3500
-$Comp
-L CP_Small C2
-U 1 1 5A971DAC
-P 1900 3100
-F 0 "C2" H 1910 3170 50  0000 L CNN
-F 1 "10uF" V 1800 3000 50  0000 L CNN
-F 2 "Capacitors_Tantalum_SMD:CP_Tantalum_Case-C_EIA-6032-28_Hand" H 1900 3100 50  0001 C CNN
-F 3 "" H 1900 3100 50  0001 C CNN
-	1    1900 3100
-	1    0    0    -1
-$EndComp
-Wire Wire Line
-	2100 3000 1900 3000
-Wire Wire Line
-	2100 3100 2100 3200
-Wire Wire Line
-	2100 3200 1900 3200
-$Comp
-L R R1
-U 1 1 5A971E49
-P 3500 3000
-F 0 "R1" V 3400 3000 50  0000 C CNN
-F 1 "20K" V 3500 3000 50  0000 C CNN
-F 2 "Resistors_SMD:R_0805_HandSoldering" V 3430 3000 50  0001 C CNN
-F 3 "" H 3500 3000 50  0001 C CNN
-	1    3500 3000
-	0    1    1    0
-$EndComp
-Wire Wire Line
-	3350 3000 3150 3000
-$Comp
-L VCC #PWR02
-U 1 1 5A971ED5
-P 2650 2250
-F 0 "#PWR02" H 2650 2100 50  0001 C CNN
-F 1 "VCC" H 2650 2400 50  0000 C CNN
-F 2 "" H 2650 2250 50  0001 C CNN
-F 3 "" H 2650 2250 50  0001 C CNN
-	1    2650 2250
-	1    0    0    -1
-$EndComp
-$Comp
-L C_Small C1
-U 1 1 5A971F06
-P 2800 2400
-F 0 "C1" H 2810 2470 50  0000 L CNN
-F 1 "2uF" H 2810 2320 50  0000 L CNN
-F 2 "Capacitors_SMD:C_0805_HandSoldering" H 2800 2400 50  0001 C CNN
-F 3 "" H 2800 2400 50  0001 C CNN
-	1    2800 2400
-	1    0    0    -1
-$EndComp
-$Comp
-L GND #PWR03
-U 1 1 5A971F51
-P 2800 2500
-F 0 "#PWR03" H 2800 2250 50  0001 C CNN
-F 1 "GND" H 2800 2350 50  0000 C CNN
-F 2 "" H 2800 2500 50  0001 C CNN
-F 3 "" H 2800 2500 50  0001 C CNN
-	1    2800 2500
-	1    0    0    -1
-$EndComp
-Wire Wire Line
-	2650 2250 2650 2600
-Wire Wire Line
-	2800 2300 2650 2300
-Connection ~ 2650 2300
-$Comp
-L R R2
-U 1 1 5A971FF1
-P 3500 3100
-F 0 "R2" V 3580 3100 50  0000 C CNN
-F 1 "102.6K" V 3500 3100 50  0000 C CNN
-F 2 "Resistors_SMD:R_0805_HandSoldering" V 3430 3100 50  0001 C CNN
-F 3 "" H 3500 3100 50  0001 C CNN
-	1    3500 3100
-	0    1    1    0
-$EndComp
-Wire Wire Line
-	3150 3100 3350 3100
-Wire Wire Line
-	2100 2900 2100 2050
-Wire Wire Line
-	2100 2050 3650 2050
-Wire Wire Line
-	3650 2050 3650 3350
-Connection ~ 3650 3000
-Wire Wire Line
-	3200 3100 3200 3550
-Wire Wire Line
-	3200 3550 4050 3550
-Connection ~ 3200 3100
-$Comp
-L CP_Small C6
-U 1 1 5A9720FC
-P 3200 3650
-F 0 "C6" H 3210 3720 50  0000 L CNN
-F 1 "100uF" H 3210 3570 50  0000 L CNN
-F 2 "Capacitors_THT:CP_Radial_D6.3mm_P2.50mm" H 3200 3650 50  0001 C CNN
-F 3 "" H 3200 3650 50  0001 C CNN
-	1    3200 3650
-	-1   0    0    1
-$EndComp
-$Comp
-L GND #PWR04
-U 1 1 5A972177
-P 3200 3800
-F 0 "#PWR04" H 3200 3550 50  0001 C CNN
-F 1 "GND" H 3200 3650 50  0000 C CNN
-F 2 "" H 3200 3800 50  0001 C CNN
-F 3 "" H 3200 3800 50  0001 C CNN
-	1    3200 3800
-	1    0    0    -1
-$EndComp
-Wire Wire Line
-	3200 3800 3200 3750
-Wire Wire Line
-	4050 3550 4050 3500
-Connection ~ 3650 3100
-$Comp
-L C_Small C5
-U 1 1 5A97221D
-P 3650 3450
-F 0 "C5" H 3660 3520 50  0000 L CNN
-F 1 "2nF" H 3800 3450 50  0000 L CNN
-F 2 "Capacitors_SMD:C_0805_HandSoldering" H 3650 3450 50  0001 C CNN
-F 3 "" H 3650 3450 50  0001 C CNN
-	1    3650 3450
-	1    0    0    -1
-$EndComp
-Connection ~ 3650 3550
 Text Notes 6300 2500 0    60   ~ 0
 LM2937
@@
 $EndComp
 $Comp
-L GND #PWR05
+L GND #PWR01
 U 1 1 5A9EEF79
 P 7100 3500
-F 0 "#PWR05" H 7100 3250 50  0001 C CNN
+F 0 "#PWR01" H 7100 3250 50  0001 C CNN
 F 1 "GND" H 7100 3350 50  0000 C CNN
 F 2 "" H 7100 3500 50  0001 C CNN
@@
 $EndComp
 $Comp
-L VCC #PWR06
+L VCC #PWR02
 U 1 1 5A9FDAE3
 P 7100 2950
-F 0 "#PWR06" H 7100 2800 50  0001 C CNN
+F 0 "#PWR02" H 7100 2800 50  0001 C CNN
 F 1 "VCC" H 7100 3100 50  0000 C CNN
 F 2 "" H 7100 2950 50  0001 C CNN
@@
 $EndComp
 $Comp
-L GND #PWR07
+L GND #PWR03
 U 1 1 5A9FDB9C
 P 6550 3500
-F 0 "#PWR07" H 6550 3250 50  0001 C CNN
+F 0 "#PWR03" H 6550 3250 50  0001 C CNN
 F 1 "GND" H 6550 3350 50  0000 C CNN
 F 2 "" H 6550 3500 50  0001 C CNN
@@
 $EndComp
 $Comp
-L GND #PWR08
+L GND #PWR04
 U 1 1 5A9FDBED
 P 6050 3500
-F 0 "#PWR08" H 6050 3250 50  0001 C CNN
+F 0 "#PWR04" H 6050 3250 50  0001 C CNN
 F 1 "GND" H 6050 3350 50  0000 C CNN
 F 2 "" H 6050 3500 50  0001 C CNN
@@
 Connection ~ 6050 3000
 $Comp
-L GND #PWR09
+L GND #PWR05
 U 1 1 5A9FDDD2
 P 5750 3300
-F 0 "#PWR09" H 5750 3050 50  0001 C CNN
+F 0 "#PWR05" H 5750 3050 50  0001 C CNN
 F 1 "GND" H 5750 3150 50  0000 C CNN
 F 2 "" H 5750 3300 50  0001 C CNN
