File: HW/Current gen.sch (KiCad schematic (older format))
At the start: 14 parts

Commit message: Add files via upload
Parts:
- removed J?: Conn_01x02_Male, Pin_Headers:Pin_Header_Straight_1x02_Pitch2.54mm_SMD_Pin1Right, symbol Conn_01x02_Male
- removed TP?: TEST, Pin_Headers:Pin_Header_Straight_1x01_Pitch2.54mm, symbol TEST
- added C? (x5): 100n, Capacitors_SMD:C_0805_HandSoldering, symbol C
- added C? (x6): C, Capacitors_SMD:C_0805_HandSoldering, symbol C
- added Q? (x2): IRFFR220N, TO_SOT_Packages_SMD:TO-252-2, symbol IRFFR220N
- added R? (x2): 10R, Resistors_THT:R_Axial_DIN0414_L11.9mm_D4.5mm_P15.24mm_Horizontal, symbol R
- added R? (x2): 0,01R, Resistors_SMD:R_2512_HandSoldering, symbol R
- added TP? (x2): TEST, Pin_Headers:Pin_Header_Straight_1x01_Pitch2.54mm, symbol TEST
- added U? (x4): OP07, Housings_DIP:DIP-8_W7.62mm_Socket_LongPads, symbol OP07
- added U? (x2): INA219, TO_SOT_Packages_SMD:SOT-23-8_Handsoldering, symbol INA219
- added U? (x2): MCP4725, TO_SOT_Packages_SMD:SOT-23-6_Handsoldering, symbol MCP4725
- C?: value C -> 100n
Connections:
- net labels added: -5V, BattV_Monitor2, BattV_Monitor3, Battery_Positive1, Battery_Positive2, Battery_Positive3
- wire segments 29 -> 75
Other:
- moved on the sheet: C?, Q?, R?, TP?, U?

Commit message: Add files via upload
Parts:
- gave numbers to parts that had none: 39

Commit message: Add files via upload
Parts:
- removed C16: 100n, Capacitors_SMD:C_0805_HandSoldering, symbol C
- removed C17, C5, C6, C7, C8: C, Capacitors_SMD:C_0805_HandSoldering, symbol C
- removed U10, U2, U3: MCP4725, TO_SOT_Packages_SMD:SOT-23-6_Handsoldering, symbol MCP4725
- removed U11, U4, U5: OP07, Housings_DIP:DIP-8_W7.62mm_Socket_LongPads, symbol OP07
- C15: value C -> 100n
Connections:
- net labels added: DAC_IN1, DAC_IN2, DAC_IN3
- net labels removed: BattV_Monitor2, BattV_Monitor3
- wire segments 75 -> 46

Commit message: Add files via upload
Parts:
- renumbered C9 to C10, C18 to C12, C14 to C13, C15 to C14, C12 to C15, C13 to C7, C19 to C8, C10 to C9, Q3 to Q2, Q2 to Q3, R7 to R4, R4 to R5, R8 to R6, R5 to R7, R6 to R8, TP3 to TP2, TP2 to TP3, U8 to U3, U13 to U4, U6 to U5, U12 to U6, U9 to U7, U7 to U8
Connections:
- net GND: now also C11.1, C12.1, C15.1
- net VCC: no longer C11.1, C12.1, C15.1

Commit message: better layout
Parts:
- removed C11, C12, C15: 100n, Capacitors_SMD:C_0805_HandSoldering, symbol C
- added C24, C25, C28: 100n, Capacitors_SMD:C_0805_HandSoldering, symbol C
- added C26, C27, C29: 1n, Capacitors_SMD:C_0805_HandSoldering, symbol C_Small
- added R27, R28, R31: 10K, Resistors_SMD:R_0805_HandSoldering, symbol R
- added R29, R30, R32: 1K, Resistors_SMD:R_0805_HandSoldering, symbol R_Small
- R5, R6, R8: footprint Resistors_THT:R_Axial_DIN0414_L11.9mm_D4.5mm_P15.24mm_Horizontal -> Resistors_SMD:R_2512_HandSoldering
Connections:
- net -5V is gone; now on net GND: U5.4 (V-), U6.4 (V-), U8.4 (V-)
- net Battery_Positive1: now also C24.1
- net Battery_Positive2: now also C25.1
- net Battery_Positive3: now also C28.1
- net DAC_IN1: now also R27.1
- net DAC_IN2: now also R28.1
- net DAC_IN3: now also R31.1
- net GND: now also R27.2, R28.2, R31.2; no longer U4.8 (ADDR1)
- net SCL: no longer U4.7 (ADDR0)
- net VCC: now also U4.7 (ADDR0), U4.8 (ADDR1)
- net B1off: now reaches Q1.1 (G), U5.6
- net B1off: now also R29.1
- net at Q1.2 (D), R3.2, U3.2 (IN-): now also C24.2
- net at Q1.3 (S), R5.1, U5.2 (-): now also C26.2
- net B3off: now reaches Q3.1 (G), U8.6
- net B3off: now also R32.1
- net at Q3.2 (D), R7.2, U7.2 (IN-): now also C28.2
- net at Q3.3 (S), R8.1, U8.2 (-): now also C29.2
- net B2off: now reaches Q2.1 (G), U6.6
- net B2off: now also R30.1
- net at Q2.2 (D), R4.2, U4.2 (IN-): now also C25.2
- net at Q2.3 (S), R6.1, U6.2 (-): now also C27.2
- new net: C27.1, R30.2
- new net: C26.1, R29.2
- new net: C29.1, R32.2
Other:
- moved on the sheet: C10, C14, C9
