File: HW/mcu.sch (KiCad schematic (older format))
At the start: 12 parts

Commit message: Add files via upload
Parts:
- added R? (x2): 1K, symbol R
Connections:
- net SCL: now also R?.2
- net SDA: now also R?.2
- net VCC: now also R?.1, R?.1
Changed lines of the file:
@@
 $Descr A4 11693 8268
 encoding utf-8
-Sheet 4 4
+Sheet 4 5
 Title ""
 Date "2017-11-18"
@@
 $EndComp
 $Comp
-L GND #PWR?
+L GND #PWR062
 U 1 1 5A97113D
 P 4800 3750
-F 0 "#PWR?" H 4800 3500 50  0001 C CNN
+F 0 "#PWR062" H 4800 3500 50  0001 C CNN
 F 1 "GND" H 4805 3577 50  0000 C CNN
 F 2 "" H 4800 3750 50  0001 C CNN
@@
 $EndComp
 $Comp
-L GND #PWR?
+L GND #PWR063
 U 1 1 5A97113E
 P 5350 5200
-F 0 "#PWR?" H 5350 4950 50  0001 C CNN
+F 0 "#PWR063" H 5350 4950 50  0001 C CNN
 F 1 "GND" H 5355 5027 50  0000 C CNN
 F 2 "" H 5350 5200 50  0001 C CNN
@@
 $EndComp
 $Comp
-L VCC #PWR?
+L VCC #PWR064
 U 1 1 5A971142
 P 1900 2800
-F 0 "#PWR?" H 1900 2650 50  0001 C CNN
+F 0 "#PWR064" H 1900 2650 50  0001 C CNN
 F 1 "VCC" H 1917 2973 50  0000 C CNN
 F 2 "" H 1900 2800 50  0001 C CNN
@@
 $EndComp
 $Comp
-L GND #PWR?
+L GND #PWR065
 U 1 1 5A971143
 P 1900 4100
-F 0 "#PWR?" H 1900 3850 50  0001 C CNN
+F 0 "#PWR065" H 1900 3850 50  0001 C CNN
 F 1 "GND" H 2150 4050 50  0000 C CNN
 F 2 "" H 1900 4100 50  0001 C CNN
@@
 $EndComp
 $Comp
-L GND #PWR?
+L GND #PWR066
 U 1 1 5A971144
 P 1550 4950
-F 0 "#PWR?" H 1550 4700 50  0001 C CNN
+F 0 "#PWR066" H 1550 4700 50  0001 C CNN
 F 1 "GND" H 1500 5100 50  0000 C CNN
 F 2 "" H 1550 4950 50  0001 C CNN
@@
 $EndComp
 $Comp
-L VCC #PWR?
+L VCC #PWR067
 U 1 1 5A971145
 P 1650 5100
-F 0 "#PWR?" H 1650 4950 50  0001 C CNN
+F 0 "#PWR067" H 1650 4950 50  0001 C CNN
 F 1 "VCC" H 1667 5273 50  0000 C CNN
 F 2 "" H 1650 5100 50  0001 C CNN
@@
 TX0
 $Comp
-L VCC #PWR?
+L VCC #PWR068
 U 1 1 5A971146
 P 5300 2550
-F 0 "#PWR?" H 5300 2400 50  0001 C CNN
+F 0 "#PWR068" H 5300 2400 50  0001 C CNN
 F 1 "VCC" H 5317 2723 50  0000 C CNN
 F 2 "" H 5300 2550 50  0001 C CNN
@@
 $EndComp
 $Comp
-L GND #PWR?
+L GND #PWR069
 U 1 1 5A97114A
 P 8450 3750
-F 0 "#PWR?" H 8450 3500 50  0001 C CNN
+F 0 "#PWR069" H 8450 3500 50  0001 C CNN
 F 1 "GND" H 8450 3600 50  0000 C CNN
 F 2 "" H 8450 3750 50  0001 C CNN
@@
 $EndComp
 $Comp
-L VCC #PWR?
+L VCC #PWR070
 U 1 1 5A97114B
 P 2650 5950
-F 0 "#PWR?" H 2650 5800 50  0001 C CNN
+F 0 "#PWR070" H 2650 5800 50  0001 C CNN
 F 1 "VCC" H 2667 6123 50  0000 C CNN
 F 2 "" H 2650 5950 50  0001 C CNN
@@
 $EndComp
 $Comp
-L GND #PWR?
+L GND #PWR071
 U 1 1 5A97114C
 P 2650 6150
-F 0 "#PWR?" H 2650 5900 50  0001 C CNN
+F 0 "#PWR071" H 2650 5900 50  0001 C CNN
 F 1 "GND" H 2600 6300 50  0000 C CNN
 F 2 "" H 2650 6150 50  0001 C CNN
@@
 $EndComp
 $Comp
-L VCC #PWR?
+L VCC #PWR072
 U 1 1 5A97114D
 P 4450 2600
-F 0 "#PWR?" H 4450 2450 50  0001 C CNN
+F 0 "#PWR072" H 4450 2450 50  0001 C CNN
 F 1 "VCC" H 4467 2773 50  0000 C CNN
 F 2 "" H 4450 2600 50  0001 C CNN
@@
 $EndComp
 $Comp
-L GND #PWR?
+L GND #PWR073
 U 1 1 5A97114E
 P 4450 2900
-F 0 "#PWR?" H 4450 2650 50  0001 C CNN
+F 0 "#PWR073" H 4450 2650 50  0001 C CNN
 F 1 "GND" H 4455 2727 50  0000 C CNN
 F 2 "" H 4450 2900 50  0001 C CNN
@@
 $EndComp
 $Comp
-L VCC #PWR?
+L VCC #PWR074
 U 1 1 5A971150
 P 4900 2600
-F 0 "#PWR?" H 4900 2450 50  0001 C CNN
+F 0 "#PWR074" H 4900 2450 50  0001 C CNN
 F 1 "VCC" H 4917 2773 50  0000 C CNN
 F 2 "" H 4900 2600 50  0001 C CNN
@@
 $EndComp
 $Comp
-L GND #PWR?
+L GND #PWR075
 U 1 1 5A971151
 P 4900 2900
-F 0 "#PWR?" H 4900 2650 50  0001 C CNN
+F 0 "#PWR075" H 4900 2650 50  0001 C CNN
 F 1 "GND" H 4905 2727 50  0000 C CNN
 F 2 "" H 4900 2900 50  0001 C CNN
@@
 	1    0    0    -1
 $EndComp
+Text GLabel 9550 2750 3    60   Input ~ 0
+SDA
+Text GLabel 9800 2750 3    60   Input ~ 0
+SCL
+$Comp
+L R R?
+U 1 1 5A972C05
+P 9550 2500
+F 0 "R?" V 9630 2500 50  0000 C CNN
+F 1 "1K" V 9550 2500 50  0000 C CNN
+F 2 "" V 9480 2500 50  0001 C CNN
+F 3 "" H 9550 2500 50  0001 C CNN
+	1    9550 2500
+	1    0    0    -1
+$EndComp
+$Comp
+L R R?
+U 1 1 5A972C5F
+P 9800 2500
+F 0 "R?" V 9880 2500 50  0000 C CNN
+F 1 "1K" V 9800 2500 50  0000 C CNN
+F 2 "" V 9730 2500 50  0001 C CNN
+F 3 "" H 9800 2500 50  0001 C CNN
+	1    9800 2500
+	1    0    0    -1
+$EndComp
+$Comp
+L VCC #PWR076
+U 1 1 5A972C9F
+P 9550 2300
+F 0 "#PWR076" H 9550 2150 50  0001 C CNN
+F 1 "VCC" H 9567 2473 50  0000 C CNN
+F 2 "" H 9550 2300 50  0001 C CNN
+F 3 "" H 9550 2300 50  0001 C CNN
+	1    9550 2300
+	1    0    0    -1
+$EndComp
+$Comp
+L VCC #PWR077
+U 1 1 5A972CD4
+P 9800 2300
+F 0 "#PWR077" H 9800 2150 50  0001 C CNN
+F 1 "VCC" H 9817 2473 50  0000 C CNN
+F 2 "" H 9800 2300 50  0001 C CNN
+F 3 "" H 9800 2300 50  0001 C CNN
+	1    9800 2300
+	1    0    0    -1
+$EndComp
+Wire Wire Line
+	9800 2300 9800 2350
+Wire Wire Line
+	9550 2300 9550 2350
+Wire Wire Line
+	9550 2650 9550 2750
+Wire Wire Line
+	9800 2650 9800 2750
 $EndSCHEMATC

Commit message: Add files via upload
Parts:
- added D1: LED1, LEDs:LED_D5.0mm-4, symbol LED_RABG
- added D2: LED2, LEDs:LED_D5.0mm-4, symbol LED_RABG
- added D3: LED3, LEDs:LED_D5.0mm-4, symbol LED_RABG
- added J1: OLED, Pin_Headers:Pin_Header_Straight_1x04_Pitch2.54mm_SMD_Pin1Left, symbol Conn_01x04
- added R18, R19, R20, R21, R22, R23, R24, R25, R26: R, Resistors_SMD:R_0805_HandSoldering, symbol R
- C21: renamed from C?; footprint (none) -> Capacitors_Tantalum_SMD:CP_Tantalum_Case-C_EIA-6032-28_Hand
- R10, R11: renamed from R?; footprint (none) -> Resistors_SMD:R_0805_HandSoldering
- gave numbers to parts that had none: 11
Connections:
- net GND: now also J1.4 (Pin_4)
- net SCL: now also J1.2 (Pin_2)
- net SDA: now also J1.1 (Pin_1)
- net VCC: now also D1.2 (A), D2.2 (A), D3.2 (A), J1.3 (Pin_3)
- net Led3G: now reaches U14.1 (3/PWM/INT1)
- net Led3G: now also R25.2
- net Led1G: now reaches U14.10 (6/PWM)
- net Led1G: now also R19.2
- net Led1B: now reaches U14.11 (7)
- net Led1B: now also R20.2
- net Led2R: now reaches U14.12 (8)
- net Led2R: now also R21.2
- net Led2G: now reaches U14.13 (9PWM)
- net Led2G: now also R22.2
- net Led2B: now reaches U14.14 (10PWM)
- net Led2B: now also R23.2
- net Led3B: now reaches U14.2 (4)
- net Led3B: now also R26.2
- net Led3R: now reaches U14.32 (2/WPM/INT0)
- net Led3R: now also R24.2
- net Led1R: now reaches U14.9 (5/PWM)
- net Led1R: now also R18.2
- new net: D1.1 (RK), R18.1
- new net: D1.3 (BK), R20.1
- new net: D1.4 (GK), R19.1
- new net: D2.1 (RK), R21.1
- new net: D2.3 (BK), R23.1
- new net: D2.4 (GK), R22.1
- new net: D3.1 (RK), R24.1
- new net: D3.3 (BK), R26.1
- new net: D3.4 (GK), R25.1
Other:
- moved on the sheet: 1U1, C20, C21, C22, C23, C24, FTDI1, ISP1, JP1, R10, R11, R9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

Commit message: Add files via upload
Parts:
- added 1U2: 0,1U, Capacitors_SMD:C_0805_HandSoldering, symbol C
- added U2: MCP4728, Housings_SSOP:MSOP-10_3x3mm_Pitch0.5mm, symbol MCP4728
Connections:
- net GND: now also 1U2.2, U2.10 (VSS), U2.4 (~LDAC)
- net SCL: now also U2.2 (SCL)
- net SDA: now also U2.3 (SDA)
- net VCC: now also 1U2.1, U2.1 (VDD)
- new net DAC_OUT1: U2.6 (VOUTA)
- new net DAC_OUT2: U2.7 (VOUTB)
- new net DAC_OUT3: U2.8 (VOUTC)
Changed lines of the file:
@@
 LIBS:contrib
 LIBS:valves
-LIBS:3-pin-boostconv
-LIBS:34063
-LIBS:Arduino
-LIBS:bluepill_breakouts
-LIBS:L298N
-LIBS:Peter-bckup
-LIBS:Peters
-LIBS:WS2812B
 LIBS:discharger-cache
 EELAYER 25 0
@@
 $EndComp
 $Comp
-L GND #PWR77
+L GND #PWR050
 U 1 1 5A97113D
 P 3500 2100
-F 0 "#PWR77" H 3500 1850 50  0001 C CNN
+F 0 "#PWR050" H 3500 1850 50  0001 C CNN
 F 1 "GND" H 3505 1927 50  0000 C CNN
 F 2 "" H 3500 2100 50  0001 C CNN
@@
 $EndComp
 $Comp
-L GND #PWR81
+L GND #PWR051
 U 1 1 5A97113E
 P 4050 3550
-F 0 "#PWR81" H 4050 3300 50  0001 C CNN
+F 0 "#PWR051" H 4050 3300 50  0001 C CNN
 F 1 "GND" H 4055 3377 50  0000 C CNN
 F 2 "" H 4050 3550 50  0001 C CNN
@@
 $EndComp
 $Comp
-L VCC #PWR71
+L VCC #PWR052
 U 1 1 5A971142
 P 1600 950
-F 0 "#PWR71" H 1600 800 50  0001 C CNN
+F 0 "#PWR052" H 1600 800 50  0001 C CNN
 F 1 "VCC" H 1617 1123 50  0000 C CNN
 F 2 "" H 1600 950 50  0001 C CNN
@@
 $EndComp
 $Comp
-L GND #PWR72
+L GND #PWR053
 U 1 1 5A971143
 P 1600 2250
-F 0 "#PWR72" H 1600 2000 50  0001 C CNN
+F 0 "#PWR053" H 1600 2000 50  0001 C CNN
 F 1 "GND" H 1850 2200 50  0000 C CNN
 F 2 "" H 1600 2250 50  0001 C CNN
@@
 $EndComp
 $Comp
-L GND #PWR69
+L GND #PWR054
 U 1 1 5A971144
 P 1250 3100
-F 0 "#PWR69" H 1250 2850 50  0001 C CNN
+F 0 "#PWR054" H 1250 2850 50  0001 C CNN
 F 1 "GND" H 1200 3250 50  0000 C CNN
 F 2 "" H 1250 3100 50  0001 C CNN
@@
 $EndComp
 $Comp
-L VCC #PWR70
+L VCC #PWR055
 U 1 1 5A971145
 P 1350 3250
-F 0 "#PWR70" H 1350 3100 50  0001 C CNN
+F 0 "#PWR055" H 1350 3100 50  0001 C CNN
 F 1 "VCC" H 1367 3423 50  0000 C CNN
 F 2 "" H 1350 3250 50  0001 C CNN
@@
 TX0
 $Comp
-L VCC #PWR80
+L VCC #PWR056
 U 1 1 5A971146
 P 4000 900
-F 0 "#PWR80" H 4000 750 50  0001 C CNN
+F 0 "#PWR056" H 4000 750 50  0001 C CNN
 F 1 "VCC" H 4017 1073 50  0000 C CNN
 F 2 "" H 4000 900 50  0001 C CNN
@@
 $EndComp
 $Comp
-L GND #PWR83
+L GND #PWR057
 U 1 1 5A97114A
 P 7150 2100
-F 0 "#PWR83" H 7150 1850 50  0001 C CNN
+F 0 "#PWR057" H 7150 1850 50  0001 C CNN
 F 1 "GND" H 7150 1950 50  0000 C CNN
 F 2 "" H 7150 2100 50  0001 C CNN
@@
 $EndComp
 $Comp
-L VCC #PWR73
+L VCC #PWR058
 U 1 1 5A97114B
 P 2350 4100
-F 0 "#PWR73" H 2350 3950 50  0001 C CNN
+F 0 "#PWR058" H 2350 3950 50  0001 C CNN
 F 1 "VCC" H 2367 4273 50  0000 C CNN
 F 2 "" H 2350 4100 50  0001 C CNN
@@
 $EndComp
 $Comp
-L GND #PWR74
+L GND #PWR059
 U 1 1 5A97114C
 P 2350 4300
-F 0 "#PWR74" H 2350 4050 50  0001 C CNN
+F 0 "#PWR059" H 2350 4050 50  0001 C CNN
 F 1 "GND" H 2300 4450 50  0000 C CNN
 F 2 "" H 2350 4300 50  0001 C CNN
@@
 $EndComp
 $Comp
-L VCC #PWR75
+L VCC #PWR060
 U 1 1 5A97114D
 P 3150 950
-F 0 "#PWR75" H 3150 800 50  0001 C CNN
+F 0 "#PWR060" H 3150 800 50  0001 C CNN
 F 1 "VCC" H 3167 1123 50  0000 C CNN
 F 2 "" H 3150 950 50  0001 C CNN
@@
 $EndComp
 $Comp
-L GND #PWR76
+L GND #PWR061
 U 1 1 5A97114E
 P 3150 1250
-F 0 "#PWR76" H 3150 1000 50  0001 C CNN
+F 0 "#PWR061" H 3150 1000 50  0001 C CNN
 F 1 "GND" H 3155 1077 50  0000 C CNN
 F 2 "" H 3150 1250 50  0001 C CNN
@@
 $EndComp
 $Comp
-L VCC #PWR78
+L VCC #PWR062
 U 1 1 5A971150
 P 3600 950
-F 0 "#PWR78" H 3600 800 50  0001 C CNN
+F 0 "#PWR062" H 3600 800 50  0001 C CNN
 F 1 "VCC" H 3617 1123 50  0000 C CNN
 F 2 "" H 3600 950 50  0001 C CNN
@@
 $EndComp
 $Comp
-L GND #PWR79
+L GND #PWR063
 U 1 1 5A971151
 P 3600 1250
-F 0 "#PWR79" H 3600 1000 50  0001 C CNN
+F 0 "#PWR063" H 3600 1000 50  0001 C CNN
 F 1 "GND" H 3605 1077 50  0000 C CNN
 F 2 "" H 3600 1250 50  0001 C CNN
@@
 $EndComp
 $Comp
-L VCC #PWR84
+L VCC #PWR064
 U 1 1 5A972C9F
 P 7900 1550
-F 0 "#PWR84" H 7900 1400 50  0001 C CNN
+F 0 "#PWR064" H 7900 1400 50  0001 C CNN
 F 1 "VCC" H 7917 1723 50  0000 C CNN
 F 2 "" H 7900 1550 50  0001 C CNN
@@
 $EndComp
 $Comp
-L VCC #PWR85
+L VCC #PWR065
 U 1 1 5A972CD4
 P 8150 1550
-F 0 "#PWR85" H 8150 1400 50  0001 C CNN
+F 0 "#PWR065" H 8150 1400 50  0001 C CNN
 F 1 "VCC" H 8167 1723 50  0000 C CNN
 F 2 "" H 8150 1550 50  0001 C CNN
@@
 SCL
 $Comp
-L VCC #PWR87
+L VCC #PWR066
 U 1 1 5A97BF05
 P 8800 1150
-F 0 "#PWR87" H 8800 1000 50  0001 C CNN
+F 0 "#PWR066" H 8800 1000 50  0001 C CNN
 F 1 "VCC" H 8800 1300 50  0000 C CNN
 F 2 "" H 8800 1150 50  0001 C CNN
@@
 $EndComp
 $Comp
-L GND #PWR88
+L GND #PWR067
 U 1 1 5A97BF37
 P 8800 1250
-F 0 "#PWR88" H 8800 1000 50  0001 C CNN
+F 0 "#PWR067" H 8800 1000 50  0001 C CNN
 F 1 "GND" H 8800 1100 50  0000 C CNN
 F 2 "" H 8800 1250 50  0001 C CNN
@@
 	5600 5650 5500 5650
 $Comp
-L VCC #PWR82
+L VCC #PWR068
 U 1 1 5A97E4AB
 P 6550 5650
-F 0 "#PWR82" H 6550 5500 50  0001 C CNN
+F 0 "#PWR068" H 6550 5500 50  0001 C CNN
 F 1 "VCC" H 6550 5800 50  0000 C CNN
 F 2 "" H 6550 5650 50  0001 C CNN
@@
 	7300 5700 7200 5700
 $Comp
-L VCC #PWR86
+L VCC #PWR069
 U 1 1 5A97EF08
 P 8250 5700
-F 0 "#PWR86" H 8250 5550 50  0001 C CNN
+F 0 "#PWR069" H 8250 5550 50  0001 C CNN
 F 1 "VCC" H 8250 5850 50  0000 C CNN
 F 2 "" H 8250 5700 50  0001 C CNN
@@
 	8850 5750 8750 5750
 $Comp
-L VCC #PWR89
+L VCC #PWR070
 U 1 1 5A97EFB2
 P 9800 5750
-F 0 "#PWR89" H 9800 5600 50  0001 C CNN
+F 0 "#PWR070" H 9800 5600 50  0001 C CNN
 F 1 "VCC" H 9800 5900 50  0000 C CNN
 F 2 "" H 9800 5750 50  0001 C CNN
@@
 Text GLabel 6000 3100 2    60   Input ~ 0
 Led3B
+$Comp
+L MCP4728 U2
+U 1 1 5A9E4E15
+P 9250 2900
+F 0 "U2" H 8750 3150 50  0000 L CNN
+F 1 "MCP4728" H 9750 3150 50  0000 R CNN
+F 2 "Housings_SSOP:MSOP-10_3x3mm_Pitch0.5mm" H 9250 2300 50  0001 C CNN
+F 3 "" H 9250 3150 50  0001 C CNN
+	1    9250 2900
+	1    0    0    -1
+$EndComp
+$Comp
+L VCC #PWR071
+U 1 1 5A9E4F9A
+P 9250 2500
+F 0 "#PWR071" H 9250 2350 50  0001 C CNN
+F 1 "VCC" H 9267 2673 50  0000 C CNN
+F 2 "" H 9250 2500 50  0001 C CNN
+F 3 "" H 9250 2500 50  0001 C CNN
+	1    9250 2500
+	1    0    0    -1
+$EndComp
+$Comp
+L GND #PWR072
+U 1 1 5A9E4FF9
+P 9250 3400
+F 0 "#PWR072" H 9250 3150 50  0001 C CNN
+F 1 "GND" H 9250 3250 50  0000 C CNN
+F 2 "" H 9250 3400 50  0001 C CNN
+F 3 "" H 9250 3400 50  0001 C CNN
+	1    9250 3400
+	1    0    0    -1
+$EndComp
+$Comp
+L C 1U2
+U 1 1 5A9E50A7
+P 9450 3650
+F 0 "1U2" H 9565 3696 50  0000 L CNN
+F 1 "0,1U" H 9565 3605 50  0000 L CNN
+F 2 "Capacitors_SMD:C_0805_HandSoldering" H 9488 3500 50  0001 C CNN
+F 3 "" H 9450 3650 50  0001 C CNN
+	1    9450 3650
+	1    0    0    -1
+$EndComp
+$Comp
+L VCC #PWR073
+U 1 1 5A9E50AD
+P 9450 3500
+F 0 "#PWR073" H 9450 3350 50  0001 C CNN
+F 1 "VCC" H 9467 3673 50  0000 C CNN
+F 2 "" H 9450 3500 50  0001 C CNN
+F 3 "" H 9450 3500 50  0001 C CNN
+	1    9450 3500
+	1    0    0    -1
+$EndComp
+$Comp
+L GND #PWR074
+U 1 1 5A9E50B3
+P 9450 3800
+F 0 "#PWR074" H 9450 3550 50  0001 C CNN
+F 1 "GND" H 9455 3627 50  0000 C CNN
+F 2 "" H 9450 3800 50  0001 C CNN
+F 3 "" H 9450 3800 50  0001 C CNN
+	1    9450 3800
+	1    0    0    -1
+$EndComp
+Wire Wire Line
+	9250 3300 9250 3400
+Wire Wire Line
+	9250 2500 9250 2600
+Text GLabel 8650 2800 0    60   Input ~ 0
+SCL
+Text GLabel 8650 2900 0    60   Input ~ 0
+SDA
+$Comp
+L GND #PWR075
+U 1 1 5A9E5343
+P 8500 3100
+F 0 "#PWR075" H 8500 2850 50  0001 C CNN
+F 1 "GND" H 8500 2950 50  0000 C CNN
+F 2 "" H 8500 3100 50  0001 C CNN
+F 3 "" H 8500 3100 50  0001 C CNN
+	1    8500 3100
+	1    0    0    -1
+$EndComp
+Wire Wire Line
+	8650 3000 8500 3000
+Wire Wire Line
+	8500 3000 8500 3100
+Wire Wire Line
+	9950 2800 9850 2800
+Wire Wire Line
+	9950 2900 9850 2900
+Wire Wire Line
+	9950 3000 9850 3000
+Text HLabel 9950 2800 2    60   Input ~ 0
+DAC_OUT1
+Text HLabel 9950 2900 2    60   Input ~ 0
+DAC_OUT2
+Text HLabel 9950 3000 2    60   Input ~ 0
+DAC_OUT3
 $EndSCHEMATC

Commit message: Add files via upload
Parts:
- renumbered C21 to C16, C20 to C17, C23 to C18, C22 to C19, C24 to C20, J1 to J2, R18 to R12, R21 to R13, R24 to R14, R19 to R15, R22 to R16, R25 to R17, R20 to R18, R23 to R19, R26 to R20, U2 to U10, U14 to U9

Commit message: Add files via upload
Connections:
- net Led1B: now also U9.10 (6/PWM); no longer U9.11 (7)
- net Led1G: now also U9.11 (7); no longer U9.10 (6/PWM)
- net Led2B: now also U9.13 (9PWM); no longer U9.14 (10PWM)
- net Led2G: now also U9.14 (10PWM); no longer U9.13 (9PWM)
- net Led3B: now also U9.1 (3/PWM/INT1); no longer U9.2 (4)
- net Led3G: now also U9.2 (4); no longer U9.1 (3/PWM/INT1)
Changed lines of the file:
@@
 Text GLabel 6000 3200 2    60   Input ~ 0
 Led1R
+Text GLabel 6000 3400 2    60   Input ~ 0
+Led1G
 Text GLabel 6000 3300 2    60   Input ~ 0
-Led1G
-Text GLabel 6000 3400 2    60   Input ~ 0
 Led1B
 Text GLabel 6000 1100 2    60   Input ~ 0
 Led2R
+Text GLabel 6000 1300 2    60   Input ~ 0
+Led2G
 Text GLabel 6000 1200 2    60   Input ~ 0
-Led2G
-Text GLabel 6000 1300 2    60   Input ~ 0
 Led2B
 Text GLabel 6000 2900 2    60   Input ~ 0
 Led3R
+Text GLabel 6000 3100 2    60   Input ~ 0
+Led3G
 Text GLabel 6000 3000 2    60   Input ~ 0
-Led3G
-Text GLabel 6000 3100 2    60   Input ~ 0
 Led3B
 $Comp

Commit message: better layout
Parts:
- added 1U3, 1U4: 0,1U, Capacitors_SMD:C_0805_HandSoldering, symbol C
- added Q7, Q8, Q9: BC847, TO_SOT_Packages_SMD:SOT-23_Handsoldering, symbol BC847
- added R33, R34, R35: 100R, Resistors_SMD:R_0805_HandSoldering, symbol R
- U10: footprint Housings_SSOP:MSOP-10_3x3mm_Pitch0.5mm -> Housings_DIP:DIP-10_W7.62mm_LongPads
Connections:
- net GND: now also 1U3.2, 1U4.2, Q7.2 (E), Q8.2 (E), Q9.2 (E)
- net VCC: now also 1U3.1, 1U4.1
- net at U9.23 (A0/14): now also R33.2
- net at U9.24 (A1/15): now also R34.2
- net at U9.25 (A2/16): now also R35.2
- new net: Q7.1 (B), R33.1
- new net: Q8.1 (B), R34.1
- new net: Q9.1 (B), R35.1
- new net B1off: Q9.3 (C)
- new net B2off: Q8.3 (C)
- new net B3off: Q7.3 (C)
Other:
- moved on the sheet: 1U1, C16

Commit message: Layout complete
Done
Parts:
- J2: footprint Pin_Headers:Pin_Header_Straight_1x04_Pitch2.54mm_SMD_Pin1Left -> Pin_Headers:Pin_Header_Straight_1x04_Pitch2.54mm
Connections:
- net MISO: no longer U9.16 (12(MISO))
- net MOSI: no longer U9.15 (11(PWM/MOSI))
- net SCK: no longer U9.17 (13(SCK))
- net at U9.23 (A0/14): no longer R33.2
- net at U9.24 (A1/15): no longer R34.2
- net at U9.25 (A2/16): no longer R35.2
- new net B1off_MCU: R35.2, U9.15 (11(PWM/MOSI))
- new net B2off_MCU: R34.2, U9.16 (12(MISO))
- new net B3off_MCU: R33.2, U9.17 (13(SCK))
Other:
- moved on the sheet: 1U2, Q7, Q8, Q9, R33, R34, R35, U10
